File: Hardware/OpenMowerMainboard/OpenMowerMainboard.kicad_pcb (KiCad board)
At the start: 2 copper layers, 242.3 x 281.6 mm, 107 parts, among them J1 Conn_02x11_Top_Bottom, J10 Conn_01x05, J11 Conn_01x03_Male, J12 Conn_01x03_Male, J13 Conn_01x03_Male, J14 Conn_01x03_Male, J15 Conn_01x02_Male, J16 Conn_02x03_Odd_Even, J17 Conn_01x02, J18 Conn_01x02, J19 Conn_01x04, J2 Conn_02x04_Top_Bottom, J3 Conn_01x02, J4 RPi_GPIO, J5 Conn_01x04, J6 Conn_01x04, J7 Conn_01x04, J8 Conn_01x04, J9 Conn_01x04, Q1 BSS138, Q10 BSS138, Q11 BSS138, Q12 BSS138, Q2 Q_PMOS_GDS, Q3 BSS138, Q4 BSS138, Q5 BSS138, Q6 Q_PMOS_GDS, Q7 BSS138, Q8 Q_PMOS_GDS, Q9 BSS138, U1 LM2596S_MODULE, U11 Pico, U12 MCP604, U13 WTV020, U3 SIP32509DT, U4 xESC2, U5 xESC2, U6 xESC2, U7 SIP32509DT, U8 MCP23S08-E/SS

Commit message: wip schematic
Parts:
- removed U8: MCP23S08-E/SS, MCP23S08-E_SS:SOP65P780X200-20N
- added D10: D_TVS, Diode_SMD:D_SMB, F.Cu at (224.5, 58.4)
- added D11: D_TVS, Diode_SMD:D_SMB, F.Cu at (224.5, 52.8)
- added D12: D_TVS, Diode_SMD:D_SMB, F.Cu at (241.2, 58.4)
- added D4: D_TVS, Diode_SMD:D_SMB, F.Cu at (224.5, 63.9)
- added D5: D_TVS, Diode_SMD:D_SMB, F.Cu at (232.8, 58.4)
- added D6: D_TVS, Diode_SMD:D_SMB, F.Cu at (232.8, 52.8)
- added D7: D_TVS, Diode_SMD:D_SMB, F.Cu at (241.2, 52.8)
- added D8: D_TVS, Diode_SMD:D_SMB, F.Cu at (241.2, 63.9)
- added D9: D_TVS, Diode_SMD:D_SMB, F.Cu at (232.8, 63.9)
- added F1: Fuse, MyModules:Fuseholder5x20_horiz_open_inline_Type-I, F.Cu at (224.1, 17.7)
- added F2: Fuse, MyModules:Fuseholder5x20_horiz_open_inline_Type-I, F.Cu at (224.1, 34.4)
- added F3: Fuse, MyModules:Fuseholder5x20_horiz_open_inline_Type-I, F.Cu at (251.4, 17.7)
- added F4: Fuse, MyModules:Fuseholder5x20_horiz_open_inline_Type-I, F.Cu at (224.1, 26.1)
- added J20: Conn_01x10_Female, Connector_PinHeader_2.54mm:PinHeader_1x10_P2.54mm_Vertical, F.Cu at (254.4, 65.4)
- added R51: R, Resistor_SMD:R_Shunt_Vishay_WSK2512_6332Metric_T2.66mm, F.Cu at (252.6, 24.3)
Connections:
- net /RobotConnectors/V_BATT_ALWAYS_ON renamed Net-(J2-Pad1)
- J2 pad 5: Net-(D2-Pad1) -> /RobotConnectors/CHARGE_SHUNT-
- J2 pad 7: V_BATT -> Net-(D3-Pad1)
- J3 pad 2: /V_CHARGE -> Net-(J3-Pad2)
- R40 pad 2: /V_CHARGE -> /RobotConnectors/V_CHARGE
- R53 pad 2: /opamps/SHUNT_CHARGE_CURRENT+ -> /RobotConnectors/CHARGE_SHUNT+
- R55 pad 2: /opamps/SHUNT_CHARGE_CURRENT- -> /RobotConnectors/CHARGE_SHUNT-

Commit message: added footprints to schematic
Parts:
- removed F1: Fuse, MyModules:Fuseholder5x20_horiz_open_inline_Type-I
- removed J16: Conn_02x03_Odd_Even, Connector_PinHeader_2.54mm:PinHeader_2x03_P2.54mm_Vertical
- removed J4: RPi_GPIO, Connector_PinSocket_2.54mm:PinSocket_2x20_P2.54mm_Vertical_SMD
- added C1: 100n, Capacitor_SMD:C_0805_2012Metric_Pad1.18x1.45mm_HandSolder, F.Cu at (-172.0, 29.1)
- added C3: 100n, Capacitor_SMD:C_0805_2012Metric_Pad1.18x1.45mm_HandSolder, F.Cu at (-176.8, 32.1)
- added C5: 100n, Capacitor_SMD:C_0805_2012Metric_Pad1.18x1.45mm_HandSolder, F.Cu at (-176.8, 29.1)
- added D1: D_Schottky, Diode_SMD:D_SOD-123F, F.Cu at (-155.1, 15.9)
- added D2: D_Schottky, Diode_SMD:D_SMA_Handsoldering, F.Cu at (-174.2, 21.1)
- added D3: D_Schottky, Diode_SMD:D_SMA_Handsoldering, F.Cu at (-174.2, 16.6)
- added J21: Raspberry_Pi_2_3, Connector_PinSocket_2.54mm:PinSocket_2x20_P2.54mm_Vertical_SMD, F.Cu at (-4.80, -78.6)
- added J22: Conn_02x03_Odd_Even, Connector_PinHeader_2.54mm:PinHeader_2x03_P2.54mm_Vertical, F.Cu at (18.3, -37.9)
- added JP1: SolderJumper_3_Bridged12, Jumper:SolderJumper-3_P1.3mm_Bridged12_Pad1.0x1.5mm, F.Cu at (-169.4, 2.20)
- added M1: Fan, Connector_JST:JST_XH_B2B-XH-A_1x02_P2.50mm_Vertical, F.Cu at (-166.1, -8.82)
- added Q13: BSS138, Package_TO_SOT_SMD:SOT-23, F.Cu at (68.4, -102.1)
- added Q14: BSS138, Package_TO_SOT_SMD:SOT-23, F.Cu at (80.5, -102.1)
- added Q15: BSS138, Package_TO_SOT_SMD:SOT-23, F.Cu at (56.3, -102.1)
- added Q16: BSS138, Package_TO_SOT_SMD:SOT-23, F.Cu at (44.2, -102.1)
- added TP1: TestPoint, TestPoint:TestPoint_Pad_D2.0mm, F.Cu at (-187.7, 6.50)
- added TP2: TestPoint, TestPoint:TestPoint_Pad_D2.0mm, F.Cu at (-179.6, 2.45)
- added TP3: TestPoint, TestPoint:TestPoint_Pad_D2.0mm, F.Cu at (-183.6, 6.50)
- added TP4: TestPoint, TestPoint:TestPoint_Pad_D2.0mm, F.Cu at (-183.6, 2.45)
- added TP5: TestPoint, TestPoint:TestPoint_Pad_D2.0mm, F.Cu at (-187.7, 2.45)
- added U10: 74HC4051, Package_SO:SSOP-16_4.4x5.2mm_P0.65mm, F.Cu at (-177.2, -8.77)
- added U9: 74HC4051, Package_SO:SSOP-16_4.4x5.2mm_P0.65mm, F.Cu at (-185.5, -8.77)
- R1, R10, R13, R14, R15, R16, R17, R18, R19, R2, R20, R21, R22, R23, R24, R25, R26, R27, R28, R29, R3, R30, R31, R4, R40, R41, R42, R43, R5, R6, R7, R8, R9: footprint Resistor_SMD:R_0805_2012Metric -> Resistor_SMD:R_0805_2012Metric_Pad1.20x1.40mm_HandSolder
- R44, R45, R46, R47, R48, R49, R50, R53, R55, R57: footprint Resistor_THT:R_Axial_DIN0309_L9.0mm_D3.2mm_P12.70mm_Horizontal -> Resistor_SMD:R_0805_2012Metric_Pad1.20x1.40mm_HandSolder
- R51: footprint Resistor_SMD:R_Shunt_Vishay_WSK2512_6332Metric_T2.66mm -> Resistor_SMD:R_2512_6332Metric_Pad1.40x3.35mm_HandSolder
Connections:
- R10 pad 1: GND -> +5V
- R10 pad 2: /RobotConnectors/HALL_SWITCH_3 -> /RobotConnectors/HALL_SWITCH_2_5V
- R15 pad 1: /RobotConnectors/HALL_SWITCH_2 -> +3V3
- R15 pad 2: /RobotConnectors/HALL_SWITCH_2_5V -> /RobotConnectors/HALL_SWITCH_3
- R16 pad 1: GND -> +5V
- R16 pad 2: /RobotConnectors/HALL_SWITCH_2 -> /RobotConnectors/HALL_SWITCH_3_5V
- R19 pad 1: /RobotConnectors/HALL_SWITCH_1 -> +3V3
- R19 pad 2: /RobotConnectors/HALL_SWITCH_1_5V -> /RobotConnectors/HALL_SWITCH_4
- R20 pad 1: GND -> +5V
- R20 pad 2: /RobotConnectors/HALL_SWITCH_1 -> /RobotConnectors/HALL_SWITCH_4_5V
- R3 pad 1: /RobotConnectors/HALL_SWITCH_4 -> +3V3
- R3 pad 2: /RobotConnectors/HALL_SWITCH_4_5V -> /RobotConnectors/HALL_SWITCH_1
- R6 pad 1: GND -> +5V
- R6 pad 2: /RobotConnectors/HALL_SWITCH_4 -> /RobotConnectors/HALL_SWITCH_1_5V
- R9 pad 1: /RobotConnectors/HALL_SWITCH_3 -> +3V3
- R9 pad 2: /RobotConnectors/HALL_SWITCH_3_5V -> /RobotConnectors/HALL_SWITCH_2
- U11 pad 1: /RaspberryPi/RXD -> /RaspberryPi/UART0_RXD
- U11 pad 10: /ESCs/ML_TX -> /pico/MUX_ADDRESS_1
- U11 pad 11: /ESCs/MC_RX -> /pico/MUX_ADDRESS_2
- U11 pad 12: /ESCs/MC_TX -> /GPS/POWER_EN
- U11 pad 14: /pico/SPI1_SCK -> /RaspberryPi/POWER_EN
- U11 pad 15: /pico/SPI1_MOSI -> /pico/SOUND_CLK
- U11 pad 16: /pico/SPI1_MISO -> /pico/SOUND_DATA
- U11 pad 17: /pico/EIO_CS -> /pico/SOUND_RESET
- U11 pad 19: /ESCs/MR_RX -> /RobotConnectors/HALL_SWITCH_1
- U11 pad 2: /RaspberryPi/TXD -> /RaspberryPi/UART0_TXD
- U11 pad 20: /ESCs/MR_TX -> /RobotConnectors/HALL_SWITCH_2
- U11 pad 21: /pico/SPI_MISO -> /IMU/MISO
- U11 pad 22: /pico/SPI0_CS -> /IMU/~{CS}
- U11 pad 24: /pico/SPI0_SCK -> /IMU/SCK
- U11 pad 25: /pico/SPI0_MOSI -> /IMU/MOSI
- U11 pad 27: /pico/LED_RX -> /RobotConnectors/HALL_SWITCH_3
- U11 pad 29: /pico/LED_TX -> /RobotConnectors/HALL_SWITCH_4
- U11 pad 34: /pico/CURRENT_CHARGE -> /CHARGE_CURRENT
- U11 pad 4: /pico/USS_TRIGGER -> /pico/MUX_OUTPUT
- U11 pad 5: /pico/USS_ECHO -> /pico/MUX_INPUT
- U11 pad 6: /GPS/RXD -> /RobotConnectors/LED_RX
- U11 pad 7: /GPS/TXD -> /RobotConnectors/LED_TX
- U11 pad 9: /ESCs/ML_RX -> /pico/MUX_ADDRESS_0
- U12 pad 12: (no net) -> unconnected-(U12-Pad12)
- U12 pad 13: (no net) -> unconnected-(U12-Pad13)
- U12 pad 14: (no net) -> unconnected-(U12-Pad14)

Commit message: wip
Parts:
- removed Q10, Q11, Q12, Q4, Q9: BSS138, Package_TO_SOT_SMD:SOT-23
- removed R1, R11, R12, R13, R14, R17, R18, R2, R21, R22, R32, R33, R34, R35, R36, R37, R38, R39, R7, R8: R, Resistor_SMD:R_0805_2012Metric_Pad1.20x1.40mm_HandSolder
- added IC1: 74ALVC164245DGG,11, 74ALVC164245DGG:SOP50P810X120-48N, F.Cu at (163.0, 74.4)
- added JP2: SolderJumper_3_Bridged12, Jumper:SolderJumper-3_P1.3mm_Bridged12_Pad1.0x1.5mm, B.Cu at (161.4, 74.4)
- added JP3: SolderJumper_3_Bridged12, Jumper:SolderJumper-3_P1.3mm_Bridged12_Pad1.0x1.5mm, B.Cu at (158.4, 74.4)
- M1: footprint Connector_JST:JST_XH_B2B-XH-A_1x02_P2.50mm_Vertical -> Connector_PinHeader_2.54mm:PinHeader_1x02_P2.54mm_Vertical; moved to B.Cu
- moved TP1 414.8 mm to (218.0, 92.8)
- moved TP2 414.8 mm to (226.1, 88.8)
- moved TP5 414.8 mm to (218.0, 88.8)
- moved C1 414.8 mm to (233.7, 115.4)
- moved C3 414.8 mm to (228.9, 118.4)
- moved C5 414.8 mm to (228.9, 115.4)
- moved TP3 414.8 mm to (222.1, 92.8)
- moved TP4 414.8 mm to (222.1, 88.8)
- moved U10 361.3 mm to (170.9, 88.0)
- moved U9 358.8 mm to (160.0, 88.0)
- moved ? 298.4 mm to (46.9, 173.3), turned to 90 degrees
- moved M1 297.2 mm to (71.1, 170.2), turned to 180 degrees
- moved J18 277.4 mm to (190.3, 56.9)
- moved J17 276.5 mm to (178.2, 56.9)
- moved ? 273.6 mm to (104.9, 173.3), turned to 90 degrees
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Connections:
- D10 pad 1: /ESCs/MR_HALL_V -> /ESCs/MR_PHASE_V
- D10 pad 2: /ESCs/MR_HALL_U -> /ESCs/MR_PHASE_U
- D11 pad 1: /ESCs/MR_HALL_W -> /ESCs/MR_PHASE_W
- D11 pad 2: /ESCs/MR_HALL_V -> /ESCs/MR_PHASE_V
- D12 pad 1: /ESCs/MR_HALL_W -> /ESCs/MR_PHASE_W
- D12 pad 2: /ESCs/MR_HALL_U -> /ESCs/MR_PHASE_U
- D4 pad 1: /ESCs/ML_HALL_V -> /ESCs/ML_PHASE_V
- D4 pad 2: /ESCs/ML_HALL_U -> /ESCs/ML_PHASE_U
- D5 pad 1: /ESCs/ML_HALL_W -> /ESCs/ML_PHASE_W
- D5 pad 2: /ESCs/ML_HALL_V -> /ESCs/ML_PHASE_V
- D6 pad 1: /ESCs/ML_HALL_W -> /ESCs/ML_PHASE_W
- D6 pad 2: /ESCs/ML_HALL_U -> /ESCs/ML_PHASE_U
- D7 pad 1: /ESCs/MC_HALL_V -> /ESCs/MC_PHASE_V
- D7 pad 2: /ESCs/MC_HALL_U -> /ESCs/MC_PHASE_U
- D8 pad 1: /ESCs/MC_HALL_W -> /ESCs/MC_PHASE_W
- D8 pad 2: /ESCs/MC_HALL_V -> /ESCs/MC_PHASE_V
- D9 pad 1: /ESCs/MC_HALL_W -> /ESCs/MC_PHASE_W
- D9 pad 2: /ESCs/MC_HALL_U -> /ESCs/MC_PHASE_U
- U10 pad 13: /RobotConnectors/USS_1_ECHO -> /RobotConnectors/USS_3_ECHO
- U10 pad 15: /RobotConnectors/USS_3_ECHO -> /RobotConnectors/USS_1_ECHO
- U11 pad 4: /pico/MUX_OUTPUT -> /pico/MUX_INPUT
- U11 pad 5: /pico/MUX_INPUT -> /pico/MUX_OUTPUT
- U9 pad 13: /RobotConnectors/USS_1_TRIGGER -> /RobotConnectors/USS_3_TRIGGER
- U9 pad 15: /RobotConnectors/USS_3_TRIGGER -> /RobotConnectors/USS_1_TRIGGER
Routing:
- net /RobotConnectors/HALL_SWITCH_3: track 0.00 -> 134.7 mm, vias 0 -> 1
- net /RobotConnectors/HALL_SWITCH_4: track 0.00 -> 105.1 mm, vias 0 -> 1
- net /RobotConnectors/HALL_SWITCH_2: track 0.00 -> 98.7 mm, vias 0 -> 1
- net /RobotConnectors/HALL_SWITCH_1: track 0.00 -> 94.6 mm, vias 0 -> 1
- net /pico/MUX_ADDRESS_0: track 0.00 -> 80.7 mm
- net /pico/MUX_ADDRESS_1: track 0.00 -> 79.1 mm
- net /pico/MUX_ADDRESS_2: track 0.00 -> 78.0 mm
- net /pico/MUX_OUTPUT: track 0.00 -> 76.7 mm, vias 0 -> 2
- net /pico/MUX_INPUT: track 0.00 -> 73.4 mm, vias 0 -> 2
- net /IMU/MOSI: track 0.00 -> 71.7 mm, vias 0 -> 1
- net /IMU/SCK: track 0.00 -> 64.1 mm
- net /IMU/MISO: track 0.00 -> 63.1 mm
- net /IMU/~{CS}: track 0.00 -> 61.5 mm
- net /RobotConnectors/HALL_SWITCH_1_5V: track 0.00 -> 52.9 mm
- net /RobotConnectors/HALL_SWITCH_2_5V: track 0.00 -> 51.2 mm
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Other:
- board size 242.3 x 281.6 mm -> 180 x 170 mm

Commit message: wip pcb layout
Parts:
- removed D3: D_Schottky, Diode_SMD:D_SMA_Handsoldering
- removed F3: Fuse, MyModules:Fuseholder5x20_horiz_open_inline_Type-I
- removed R53, R55: 1k5, Resistor_SMD:R_0805_2012Metric_Pad1.20x1.40mm_HandSolder
- removed R57: 27k, Resistor_SMD:R_0805_2012Metric_Pad1.20x1.40mm_HandSolder
- removed TP3, TP4: TestPoint, TestPoint:TestPoint_Pad_D2.0mm
- removed U12: MCP604, Package_SO:SOIC-14_3.9x8.7mm_P1.27mm
- added C2: C_Polarized, Capacitor_THT:CP_Radial_D10.0mm_P5.00mm, F.Cu at (36.3, 124.0)
- added C4: C_Polarized, Capacitor_THT:CP_Radial_D10.0mm_P5.00mm, F.Cu at (101.3, 124.0)
- added C6: C_Polarized, Capacitor_THT:CP_Radial_D10.0mm_P5.00mm, F.Cu at (30.3, 124.0)
- added C7: C_Polarized, Capacitor_THT:CP_Radial_D10.0mm_P5.00mm, F.Cu at (68.8, 124.0)
- added C8: C_Polarized, Capacitor_THT:CP_Radial_D10.0mm_P5.00mm, F.Cu at (95.3, 124.0)
- added D13: D_Schottky, Diode_SMD:D_SOD-123F, F.Cu at (134.2, 105.2)
- added D14: D_Zener, Diode_SMD:D_SOD-123F, F.Cu at (134.2, 107.8)
- added IC2: TSC101CILT, TSC101CILT:SOT95P280X145-5N, F.Cu at (134.2, 101.2)
- added U2: MCP604, Package_SO:SOIC-14_3.9x8.7mm_P1.27mm, F.Cu at (188.3, 71.7)
- C3: value 100n -> C_Polarized; footprint Capacitor_SMD:C_0805_2012Metric_Pad1.18x1.45mm_HandSolder -> Capacitor_THT:CP_Radial_D10.0mm_P5.00mm
- JP1: moved to B.Cu
- moved D1 363.3 mm to (167.0, 184.0), turned to -90 degrees
- moved JP1 328.3 mm to (154.0, 58.8), turned to 180 degrees
- moved Q3 301.3 mm to (163.0, 184.0)
- moved R5 295.1 mm to (159.0, 184.0), turned to -90 degrees
- moved R4 290.9 mm to (156.0, 184.0), turned to 90 degrees
- moved D2 272.2 mm to (95.6, 57.2)
- moved R40 242.6 mm to (131.8, 57.4), turned to 180 degrees
- moved U7 241.0 mm to (154.0, 58.9), turned to 90 degrees
- moved R42 240.4 mm to (131.8, 59.6), turned to 180 degrees
- moved R41 239.7 mm to (136.0, 57.4), turned to 180 degrees
- moved R43 237.6 mm to (136.0, 59.6), turned to 180 degrees
- moved U3 184.7 mm to (121.5, 183.4), turned to -90 degrees
- moved C3 166.1 mm to (62.8, 124.0), turned to 180 degrees
- moved R29 139.8 mm to (70.8, 140.1), turned to -90 degrees
- moved R26 139.1 mm to (103.3, 140.1), turned to -90 degrees
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Connections:
- C1 pad 1: Net-(C1-Pad1) -> +5V
- C1 pad 2: /RobotConnectors/CHARGE_SHUNT- -> GND
- C3 pad 1: /CHARGE_CURRENT -> /ESCs/MOSFET_SWITCH2/VOUT
- C3 pad 2: Net-(C3-Pad2) -> GND
- J15 pad 2: Net-(F3-Pad1) -> Net-(F2-Pad2)
- U11 pad 10: /pico/MUX_ADDRESS_1 -> /RobotConnectors/HALL_SWITCH_1
- U11 pad 11: /pico/MUX_ADDRESS_2 -> /pico/SOUND_CLK
- U11 pad 12: /GPS/POWER_EN -> /pico/SOUND_DATA
- U11 pad 14: /RaspberryPi/POWER_EN -> /pico/SOUND_RESET
- U11 pad 15: /pico/SOUND_CLK -> /pico/MUX_INPUT
- U11 pad 16: /pico/SOUND_DATA -> /pico/MUX_OUTPUT
- U11 pad 17: /pico/SOUND_RESET -> /pico/MUX_ADDRESS_0
- U11 pad 19: /RobotConnectors/HALL_SWITCH_1 -> /pico/MUX_ADDRESS_1
- U11 pad 20: /RobotConnectors/HALL_SWITCH_2 -> /pico/MUX_ADDRESS_2
- U11 pad 27: /RobotConnectors/HALL_SWITCH_3 -> /RaspberryPi/POWER_EN
- U11 pad 29: /RobotConnectors/HALL_SWITCH_4 -> /GPS/POWER_EN
- U11 pad 4: /pico/MUX_INPUT -> /RobotConnectors/HALL_SWITCH_4
- U11 pad 5: /pico/MUX_OUTPUT -> /RobotConnectors/HALL_SWITCH_3
- U11 pad 9: /pico/MUX_ADDRESS_0 -> /RobotConnectors/HALL_SWITCH_2
Routing:
- net +5V: track 0.00 -> 898.1 mm, vias 0 -> 9
- net V_BATT: track 0.00 -> 260.2 mm
- net +3V3: track 12.3 -> 254.3 mm, vias 0 -> 13
- net /ESCs/MC_POWER: track 0.00 -> 176.3 mm, vias 0 -> 2
- net /ESCs/ML_RX: track 0.00 -> 169.4 mm, vias 0 -> 1
- net /ESCs/ML_TX: track 0.00 -> 159.7 mm, vias 0 -> 1
- net /RaspberryPi/PICO_SWCLK: track 0.00 -> 156.5 mm, vias 0 -> 1
- net /ESCs/MC_RX: track 0.00 -> 154.3 mm, vias 0 -> 1
- net /RaspberryPi/UART0_RXD: track 0.00 -> 154.2 mm
- net /RaspberryPi/PICO_SWDIO: track 0.00 -> 152.1 mm
- net /RaspberryPi/UART0_TXD: track 0.00 -> 149.1 mm
- net /pico/SOUND_CLK: track 0.00 -> 142.8 mm, vias 0 -> 2
- net /pico/SOUND_RESET: track 0.00 -> 142.6 mm, vias 0 -> 2
- net /ESCs/MC_TX: track 0.00 -> 140.8 mm, vias 0 -> 1
- net /RaspberryPi/POWER_EN: track 0.00 -> 132.3 mm, vias 0 -> 1
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- added copper zone on B.Cu, net +5V
- added copper zone on F.Cu, net +5V
- added copper zone on F.Cu, net /RaspberryPi/RASPI_POWER
- added copper zone on F.Cu, net V_BATT
Other:
- outline, holes or cut-outs redrawn

Commit message: routing mostly done
Connections:
- net /RobotConnectors/CHARGE_SHUNT+ renamed /RobotConnectors/CHARGE_SHUNT_PLUS
- net /RobotConnectors/CHARGE_SHUNT- renamed /RobotConnectors/CHARGE_SHUNT_MINUS
- net /RobotConnectors/SPEAKER+ renamed /RobotConnectors/SPEAKER_PLUS
- net /RobotConnectors/SPEAKER- renamed /RobotConnectors/SPEAKER_MINUS
Routing:
- net /RobotConnectors/SPEAKER_MINUS: track 0.00 -> 215.2 mm, vias 0 -> 4
- net /RobotConnectors/SPEAKER_PLUS: track 0.00 -> 210.6 mm, vias 0 -> 3
- net +3V3: track 254.3 -> 409.3 mm, vias 13 -> 17
- net +5V: track 898.1 -> 924.6 mm, vias 9 -> 12
- net Net-(U4-Pad2): track 90.4 -> 82.1 mm
- net /ESCs/MOSFET_SWITCH2/VOUT: track 90.0 -> 95.0 mm
- net /ESCs/MOSFET_SWITCH1/VOUT: track 90.7 -> 95.7 mm
- net /ESCs/MOSFET_SWITCH/VOUT: track 90.0 -> 95.0 mm
- net /pico/SOUND_RESET: track 142.6 -> 146.2 mm
- net /RobotConnectors/HALL_SWITCH_4_5V: track 25.5 -> 28.8 mm
- net /RobotConnectors/HALL_SWITCH_3_5V: track 34.7 -> 38.0 mm
- net /RobotConnectors/HALL_SWITCH_2_5V: track 47.2 -> 50.4 mm
- net /RobotConnectors/HALL_SWITCH_1_5V: track 59.6 -> 62.8 mm
- net /RobotConnectors/HALL_SWITCH_3: track 23.3 -> 26.4 mm
- net /RobotConnectors/HALL_SWITCH_1: track 18.9 -> 22.0 mm
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