File: Hardware/OpenMowerMainboard/OpenMowerMainboard.kicad_pcb (KiCad board)
At the start: 2 copper layers, 180 x 170 mm, 118 parts, among them IC1 74ALVC164245DGG,11, IC2 TSC101CILT, J1 Conn_02x11_Top_Bottom, J10 Conn_01x05, J11 Conn_01x03_Male, J12 Conn_01x03_Male, J13 Conn_01x03_Male, J14 Conn_01x03_Male, J15 Conn_01x02_Male, J17 Conn_01x02, J18 Conn_01x02, J19 Conn_01x04, J2 Conn_02x04_Top_Bottom, J20 Conn_01x10_Female, J21 Raspberry_Pi_2_3, J22 Conn_02x03_Odd_Even, J3 Conn_01x02, J5 Conn_01x04, J6 Conn_01x04, J7 Conn_01x04, J8 Conn_01x04, J9 Conn_01x04, M1 Fan, Q1 BSS138, Q13 BSS138, Q14 BSS138, Q15 BSS138, Q16 BSS138, Q2 Q_PMOS_GDS, Q3 BSS138, Q5 BSS138, Q6 Q_PMOS_GDS, Q7 BSS138, Q8 Q_PMOS_GDS, U1 LM2596S_MODULE, U10 74HC4051, U11 Pico, U13 WTV020, U2 MCP604, U3 SIP32509DT, U4 xESC2, U5 xESC2, U6 xESC2, U7 SIP32509DT, U9 74HC4051

Commit message: v1.0 release candidate
Parts:
- added G***: LOGO, x-tech-logo:x-tech-logo, F.Cu at (43.6, 178.9)
- added REF**: ESD-Logo_6.6x6mm_SilkScreen, Symbol:ESD-Logo_6.6x6mm_SilkScreen, F.Cu at (35.9, 178.6)
Routing:
- net /ESCs/ML_PHASE_V: track 41.2 -> 35.3 mm
- net /ESCs/MC_PHASE_U: track 53.1 -> 48.0 mm
- net /ESCs/ML_PHASE_U: track 45.6 -> 40.5 mm
- net /ESCs/MC_PHASE_W: track 48.3 -> 43.2 mm
- net /ESCs/MC_PHASE_V: track 47.0 -> 44.5 mm
- net /RobotConnectors/SPEAKER_MINUS: track 215.2 -> 216.5 mm
- net +3V3: track 409.3 -> 410.3 mm
- net /RaspberryPi/UART0_RXD: track 154.4 -> 155.3 mm
- net +5V: track 924.6 -> 924.0 mm
- net GND: vias 364 -> 379
- added copper zone on B.Cu, net /ESCs/MC_PHASE_U
- added copper zone on F.Cu, net /ESCs/MC_PHASE_U
- added copper zone on B.Cu, net /ESCs/MC_PHASE_V
- added copper zone on F.Cu, net /ESCs/MC_PHASE_V
- added copper zone on B.Cu, net /ESCs/MC_PHASE_W
- added copper zone on F.Cu, net /ESCs/MC_PHASE_W
- added copper zone on B.Cu, net /ESCs/ML_PHASE_U
- added copper zone on F.Cu, net /ESCs/ML_PHASE_U
- added copper zone on B.Cu, net /ESCs/ML_PHASE_V
- added copper zone on F.Cu, net /ESCs/ML_PHASE_V
- added copper zone on B.Cu, net /ESCs/ML_PHASE_W
- added copper zone on F.Cu, net /ESCs/ML_PHASE_W
- added copper zone on B.Cu, net /ESCs/MR_PHASE_U
- added copper zone on F.Cu, net /ESCs/MR_PHASE_U
- added copper zone on B.Cu, net /ESCs/MR_PHASE_V
- added copper zone on F.Cu, net /ESCs/MR_PHASE_V
- added copper zone on B.Cu, net /ESCs/MR_PHASE_W
- added copper zone on F.Cu, net /ESCs/MR_PHASE_W
Other:
- board text added: "3.3V"
- board text added: "5V"
- board text added: "5V,TRIG,ECHO,GND"
- board text added: "Busy"
- board text added: "Charge"
- board text added: "Clock"
- board text added: "Data"
- board text added: "GND"
- board text added: "GND,SIG,5V"
- board text added: "Hall 1"
- board text added: "Hall 2"
- board text added: "Hall 3"
- board text added: "Hall 4"
- board text added: "IOREF"
- board text added: "Motor Connection"
- board text added: "Mower Hall Sensors"
- board text added: "OpenMower Mainboard v1.0 License CC BY-NC-SA 4.0 https://github.com/ClemensElflein/OpenMower"
- board text added: "Power Connection"
- board text added: "RXD"
- board text added: "Rain"
- board text added: "Reset"
- board text added: "Speaker"
- board text added: "Speaker +"
- board text added: "Speaker -"
- board text added: "TXD"
- board text added: "UI Board"
- board text added: "USS 1"
- board text added: "USS 2"
- board text added: "USS 3"
- board text added: "USS 4"
- board text added: "USS 5"
- board text added: "xESC Center"
- board text added: "xESC Left"
- board text added: "xESC Right"

Commit message: ordered
Other:
- board text added: "JLCJLCJLCJLC"
