File: Hardware/OpenMowerMainboard/mosfet_switch.kicad_sch (KiCad schematic)
At the start: 5 parts, among them Q5 BSS138, Q6 Q_PMOS_GDS

Commit message: wip
Parts:
- renumbered Q5 to Q7, Q6 to Q8, R26 to R29, R27 to R30, R28 to R31
Changed lines of the file:
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@@
   (symbol (lib_id "Device:R") (at 107.95 97.79 0)
     (in_bom yes) (on_board yes) (fields_autoplaced)
-    (property "Reference" "R26" (id 0) (at 110.49 96.5199 0)
+    (property "Reference" "R29" (id 0) (at 110.49 96.5199 0)
       (effects (font (size 1.27 1.27)) (justify left))
     )
@@
   (symbol (lib_id "Device:R") (at 114.3 90.17 90)
     (in_bom yes) (on_board yes) (fields_autoplaced)
-    (property "Reference" "R27" (id 0) (at 114.3 83.82 90))
+    (property "Reference" "R30" (id 0) (at 114.3 83.82 90))
     (property "Value" "R" (id 1) (at 114.3 86.36 90))
     (property "Footprint" "Resistor_SMD:R_0805_2012Metric_Pad1.20x1.40mm_HandSolder" (id 2) (at 114.3 91.948 90)
@@
   (symbol (lib_id "Device:Q_PMOS_GDS") (at 135.89 80.01 0)
     (in_bom yes) (on_board yes) (fields_autoplaced)
-    (property "Reference" "Q6" (id 0) (at 142.24 78.7399 0)
+    (property "Reference" "Q8" (id 0) (at 142.24 78.7399 0)
       (effects (font (size 1.27 1.27)) (justify left))
     )
@@
   (symbol (lib_id "Transistor_FET:BSS138") (at 125.73 90.17 0)
     (in_bom yes) (on_board yes) (fields_autoplaced)
-    (property "Reference" "Q5" (id 0) (at 132.08 88.8999 0)
+    (property "Reference" "Q7" (id 0) (at 132.08 88.8999 0)
       (effects (font (size 1.27 1.27)) (justify left))
     )
@@
   (symbol (lib_id "Device:R") (at 128.27 71.12 0)
     (in_bom yes) (on_board yes) (fields_autoplaced)
-    (property "Reference" "R28" (id 0) (at 130.81 69.8499 0)
+    (property "Reference" "R31" (id 0) (at 130.81 69.8499 0)
       (effects (font (size 1.27 1.27)) (justify left))
     )

Commit message: wip pcb layout
Parts:
- renumbered Q7 to Q5, Q8 to Q6, R29 to R26, R30 to R27, R31 to R28
Changed lines of the file:
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@@
   (symbol (lib_id "Device:R") (at 107.95 97.79 0)
     (in_bom yes) (on_board yes) (fields_autoplaced)
-    (property "Reference" "R29" (id 0) (at 110.49 96.5199 0)
+    (property "Reference" "R26" (id 0) (at 110.49 96.5199 0)
       (effects (font (size 1.27 1.27)) (justify left))
     )
@@
   (symbol (lib_id "Device:R") (at 114.3 90.17 90)
     (in_bom yes) (on_board yes) (fields_autoplaced)
-    (property "Reference" "R30" (id 0) (at 114.3 83.82 90))
+    (property "Reference" "R27" (id 0) (at 114.3 83.82 90))
     (property "Value" "R" (id 1) (at 114.3 86.36 90))
     (property "Footprint" "Resistor_SMD:R_0805_2012Metric_Pad1.20x1.40mm_HandSolder" (id 2) (at 114.3 91.948 90)
@@
   (symbol (lib_id "power:GND") (at 118.11 111.76 0)
     (in_bom yes) (on_board yes)
-    (property "Reference" "#PWR0126" (id 0) (at 118.11 118.11 0)
+    (property "Reference" "#PWR0125" (id 0) (at 118.11 118.11 0)
       (effects (font (size 1.27 1.27)) hide)
     )
@@
   (symbol (lib_id "Device:Q_PMOS_GDS") (at 135.89 80.01 0)
     (in_bom yes) (on_board yes) (fields_autoplaced)
-    (property "Reference" "Q8" (id 0) (at 142.24 78.7399 0)
+    (property "Reference" "Q6" (id 0) (at 142.24 78.7399 0)
       (effects (font (size 1.27 1.27)) (justify left))
     )
@@
   (symbol (lib_id "Transistor_FET:BSS138") (at 125.73 90.17 0)
     (in_bom yes) (on_board yes) (fields_autoplaced)
-    (property "Reference" "Q7" (id 0) (at 132.08 88.8999 0)
+    (property "Reference" "Q5" (id 0) (at 132.08 88.8999 0)
       (effects (font (size 1.27 1.27)) (justify left))
     )
@@
   (symbol (lib_id "Device:R") (at 128.27 71.12 0)
     (in_bom yes) (on_board yes) (fields_autoplaced)
-    (property "Reference" "R31" (id 0) (at 130.81 69.8499 0)
+    (property "Reference" "R28" (id 0) (at 130.81 69.8499 0)
       (effects (font (size 1.27 1.27)) (justify left))
     )
