File: Hardware/OpenMowerMainboard/mosfet_switch.kicad_sch (KiCad schematic)
At the start: 5 parts, among them Q5 BSS138, Q6 Q_PMOS_GDS

Commit message: feat(bom): update LCSC codes
Parts:
- Q5: LCSC C360338 -> C3040446
- Q6: LCSC (none) -> C26340
- R26, R28: LCSC (none) -> C17414
- R27: LCSC (none) -> C114523
Changed lines of the file:
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@@
+      (effects (font (size 1.27 1.27)) hide)
+    )
+    (property "LCSC" "C17414" (id 7) (at 107.95 97.79 0)
       (effects (font (size 1.27 1.27)) hide)
     )
@@
     )
     (property "Part Number" "RC0805FR-07150RL" (id 6) (at 114.3 90.17 0)
+      (effects (font (size 1.27 1.27)) hide)
+    )
+    (property "LCSC" "C114523" (id 7) (at 114.3 90.17 0)
       (effects (font (size 1.27 1.27)) hide)
     )
@@
       (effects (font (size 1.27 1.27)) hide)
     )
+    (property "LCSC" "C26340" (id 7) (at 135.89 80.01 0)
+      (effects (font (size 1.27 1.27)) hide)
+    )
     (pin "1")
     (pin "2")
@@
       (effects (font (size 1.27 1.27)) (justify left) hide)
     )
-    (property "LCSC" "C360338" (id 4) (at 125.73 90.17 0)
+    (property "LCSC" "C3040446" (id 4) (at 125.73 90.17 0)
       (effects (font (size 1.27 1.27)) hide)
     )
@@
       (effects (font (size 1.27 1.27)) hide)
     )
+    (property "LCSC" "C17414" (id 7) (at 128.27 71.12 0)
+      (effects (font (size 1.27 1.27)) hide)
+    )
