File: Hardware/OpenMowerMainboard/IMU.kicad_sch (KiCad schematic)
At the start: 1 part, among them J11 Conn_01x10_Female

Commit message: wip schematic
Parts:
- renumbered J11 to J20
Changed lines of the file:
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@@
   (symbol (lib_id "Connector:Conn_01x10_Female") (at 162.56 66.04 0) (unit 1)
     (in_bom yes) (on_board yes)
-    (property "Reference" "J11" (id 0) (at 163.2712 66.6496 0)
+    (property "Reference" "J20" (id 0) (at 163.2712 66.6496 0)
       (effects (font (size 1.27 1.27)) (justify left))
     )

Commit message: BoM data added to kicad - results exported to .xlsx file
Parts:
- J20: LCSC (none) -> C2894933; Part Number (none) -> PZ254-1-10-Z-8.5; Stock_PN (none) -> J-TH-1x10-.1
Changed lines of the file:
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@@
+      (effects (font (size 1.27 1.27)) hide)
+    )
+    (property "LCSC" "C2894933" (id 4) (at 162.56 66.04 0)
+      (effects (font (size 1.27 1.27)) hide)
+    )
+    (property "Part Number" "	PZ254-1-10-Z-8.5" (id 5) (at 162.56 66.04 0)
+      (effects (font (size 1.27 1.27)) hide)
+    )
+    (property "Stock_PN" "J-TH-1x10-.1" (id 6) (at 162.56 66.04 0)
       (effects (font (size 1.27 1.27)) hide)
     )
