File: Hardware/OpenMowerMainboard/RobotConnectors.kicad_sch (KiCad schematic)
At the start: 27 parts, among them IC1 74ALVC164245DGG,11, J1 Conn_02x11_Top_Bottom, J10 Conn_01x05, J11 Conn_01x03_Male, J12 Conn_01x03_Male, J13 Conn_01x03_Male, J14 Conn_01x03_Male, J17 Conn_01x02, J18 Conn_01x02, J19 Conn_01x04, J2 Conn_02x04_Top_Bottom, J3 Conn_01x02, J4 Conn_01x05, J5 Conn_01x04, J6 Conn_01x04, J7 Conn_01x04, J8 Conn_01x04, J9 Conn_01x04

Commit message: Fuse holders and aternative led led pn from lcsc added
Parts:
- F2, F4: Digikey (none) -> FC-202-24-ND; Part Number (none) -> FC-202-24; Stock_PN (none) -> FH-FC-202-24
Changed lines of the file:
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@@
+      (effects (font (size 1.27 1.27)) hide)
+    )
+    (property "Digikey" "FC-202-24-ND" (id 4) (at 118.745 68.58 0)
+      (effects (font (size 1.27 1.27)) hide)
+    )
+    (property "Part Number" "FC-202-24" (id 5) (at 118.745 68.58 0)
+      (effects (font (size 1.27 1.27)) hide)
+    )
+    (property "Stock_PN" "FH-FC-202-24" (id 6) (at 118.745 68.58 0)
       (effects (font (size 1.27 1.27)) hide)
     )
@@
       (effects (font (size 1.27 1.27)) hide)
     )
+    (property "Digikey" "FC-202-24-ND" (id 4) (at 94.615 33.02 0)
+      (effects (font (size 1.27 1.27)) hide)
+    )
+    (property "Part Number" "FC-202-24" (id 5) (at 94.615 33.02 0)
+      (effects (font (size 1.27 1.27)) hide)
+    )
+    (property "Stock_PN" "FH-FC-202-24" (id 6) (at 94.615 33.02 0)
+      (effects (font (size 1.27 1.27)) hide)
+    )

Commit message: BOM changes
Parts:
- JP2, JP3: DNP (none) -> Y
Changed lines of the file:
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@@
+      (effects (font (size 1.27 1.27)) hide)
+    )
+    (property "DNP" "Y" (id 5) (at 128.905 95.25 0)
       (effects (font (size 1.27 1.27)) hide)
     )
@@
       (effects (font (size 1.27 1.27)) hide)
     )
+    (property "DNP" "Y" (id 5) (at 161.29 172.085 0)
+      (effects (font (size 1.27 1.27)) hide)
+    )

Commit message: temporary fix - fuse holder PN
Parts:
- F2, F4: Digikey FC-202-24-ND -> (none); Part Number FC-202-24 -> https://fr.aliexpress.com/item/4000318714025.html?spm=a2g0o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; Stock_PN FH-FC-202-24 -> (none)
Changed lines of the file:
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@@
       (effects (font (size 1.27 1.27)) hide)
     )
-    (property "Digikey" "FC-202-24-ND" (id 4) (at 118.745 68.58 0)
-      (effects (font (size 1.27 1.27)) hide)
-    )
-    (property "Part Number" "FC-202-24" (id 5) (at 118.745 68.58 0)
-      (effects (font (size 1.27 1.27)) hide)
-    )
-    (property "Stock_PN" "FH-FC-202-24" (id 6) (at 118.745 68.58 0)
+    (property "Digikey" "" (id 4) (at 118.745 68.58 0)
+      (effects (font (size 1.27 1.27)) hide)
+    )
+    (property "Part Number" "https://fr.aliexpress.com/item/4000318714025.html?spm=a2g0o.order_list.0.0.70135e5bZBlpBc&gatewayAdapt=glo2fra" (id 5) (at 118.745 68.58 0)
+      (effects (font (size 1.27 1.27)) hide)
+    )
+    (property "Stock_PN" "" (id 6) (at 118.745 68.58 0)
       (effects (font (size 1.27 1.27)) hide)
     )
@@
       (effects (font (size 1.27 1.27)) hide)
     )
-    (property "Digikey" "FC-202-24-ND" (id 4) (at 94.615 33.02 0)
-      (effects (font (size 1.27 1.27)) hide)
-    )
-    (property "Part Number" "FC-202-24" (id 5) (at 94.615 33.02 0)
-      (effects (font (size 1.27 1.27)) hide)
-    )
-    (property "Stock_PN" "FH-FC-202-24" (id 6) (at 94.615 33.02 0)
-      (effects (font (size 1.27 1.27)) hide)
-    )
+    (property "Digikey" "" (id 4) (at 94.615 33.02 0)
+      (effects (font (size 1.27 1.27)) hide)
+    )
+    (property "Part Number" "https://fr.aliexpress.com/item/4000318714025.html?spm=a2g0o.order_list.0.0.70135e5bZBlpBc&gatewayAdapt=glo2fra" (id 5) (at 94.615 33.02 0)
+      (effects (font (size 1.27 1.27)) hide)
+    )
+    (property "Stock_PN" "" (id 6) (at 94.615 33.02 0)
+      (effects (font (size 1.27 1.27)) hide)
+    )
