File: Hardware/OpenMowerMainboard/opamps.kicad_sch (KiCad schematic)
At the start: 16 parts, among them IC2 TSC101CILT, U2 MCP604

Commit message: feat(bom): update LCSC codes
Parts:
- C1, C5: LCSC (none) -> C85866
- R44, R46: LCSC (none) -> C126351
- R45, R47: LCSC (none) -> C95781
- R48, R50: LCSC (none) -> C17414
- R49: LCSC (none) -> C60816
Changed lines of the file:
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@@
+      (effects (font (size 1.27 1.27)) hide)
+    )
+    (property "LCSC" "C85866" (id 7) (at 163.195 164.465 0)
       (effects (font (size 1.27 1.27)) hide)
     )
@@
       (effects (font (size 1.27 1.27)) hide)
     )
+    (property "LCSC" "C60816" (id 7) (at 100.33 78.74 0)
+      (effects (font (size 1.27 1.27)) hide)
+    )
     (pin "1")
     (pin "2")
@@
       (effects (font (size 1.27 1.27)) hide)
     )
+    (property "LCSC" "C95781" (id 7) (at 92.71 67.31 0)
+      (effects (font (size 1.27 1.27)) hide)
+    )
     (pin "1")
     (pin "2")
@@
       (effects (font (size 1.27 1.27)) hide)
     )
+    (property "LCSC" "C17414" (id 7) (at 100.33 58.42 0)
+      (effects (font (size 1.27 1.27)) hide)
+    )
     (pin "1")
     (pin "2")
@@
     )
     (property "Part Number" "RC0805FR-0747KL" (id 6) (at 49.53 76.2 0)
+      (effects (font (size 1.27 1.27)) hide)
+    )
+    (property "LCSC" "C126351" (id 7) (at 49.53 76.2 0)
       (effects (font (size 1.27 1.27)) hide)
     )
@@
       (effects (font (size 1.27 1.27)) hide)
     )
+    (property "LCSC" "C126351" (id 7) (at 74.93 81.28 0)
+      (effects (font (size 1.27 1.27)) hide)
+    )
     (pin "1")
     (pin "2")
@@
       (effects (font (size 1.27 1.27)) hide)
     )
+    (property "LCSC" "C17414" (id 7) (at 111.76 53.34 0)
+      (effects (font (size 1.27 1.27)) hide)
+    )
     (pin "1")
     (pin "2")
@@
     )
     (property "Part Number" "RC0805FR-071KL" (id 6) (at 59.69 81.28 0)
+      (effects (font (size 1.27 1.27)) hide)
+    )
+    (property "LCSC" "C95781" (id 7) (at 59.69 81.28 0)
       (effects (font (size 1.27 1.27)) hide)
     )
@@
       (effects (font (size 1.27 1.27)) hide)
     )
+    (property "LCSC" "C85866" (id 7) (at 213.995 128.27 0)
+      (effects (font (size 1.27 1.27)) hide)
+    )
